File: HuntsmanElite.kicad_sch (KiCad schematic)
At the start: 1 part, among them U1 ATmega32U4-A

Commit message: .
Connections:
- net +5V: now reaches U1.14 (VCC), U1.34 (VCC)
- net +5V: now also U1.2 (UVCC), U1.24 (AVCC), U1.44 (AVCC)
- net GND: now reaches U1.15 (GND), U1.23 (GND), U1.35 (GND), U1.43 (GND)
- net GND: now also U1.5 (UGND)
Changed lines of the file:
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@@
 (kicad_sch (version 20230121) (generator eeschema)
   (paper "A4")
+  (junction (at 82.55 30.48) (diameter 0) (color 0 0 0 0)
+  )
+  (junction (at 82.55 34.29) (diameter 0) (color 0 0 0 0)
+  )
+  (junction (at 82.55 125.73) (diameter 0) (color 0 0 0 0)
+  )
+  (junction (at 85.09 34.29) (diameter 0) (color 0 0 0 0)
+  )
+  (wire (pts (xy 82.55 30.48) (xy 82.55 34.29))
+    (stroke (width 0) (type default))
+  )
+  (wire (pts (xy 82.55 125.73) (xy 85.09 125.73))
+    (stroke (width 0) (type default))
+  )
+  (wire (pts (xy 85.09 34.29) (xy 87.63 34.29))
+    (stroke (width 0) (type default))
+  )
+  (wire (pts (xy 82.55 29.21) (xy 82.55 30.48))
+    (stroke (width 0) (type default))
+  )
+  (wire (pts (xy 82.55 34.29) (xy 85.09 34.29))
+    (stroke (width 0) (type default))
+  )
+  (wire (pts (xy 76.2 125.73) (xy 82.55 125.73))
+    (stroke (width 0) (type default))
+  )
   (symbol (lib_id "MCU_Microchip_ATmega:ATmega32U4-A") (at 85.09 80.01 0) (unit 1)
     (in_bom yes) (on_board yes) (dnp no) (fields_autoplaced)
@@
         )
       )
+    )
+  )
+  (symbol (lib_id "power:+5V") (at 82.55 30.48 0) (unit 1)
+    (in_bom yes) (on_board yes) (dnp no) (fields_autoplaced)
+    (property "Reference" "#PWR01" (at 82.55 34.29 0)
+      (effects (font (size 1.27 1.27)) hide)
+    )
+    (property "Value" "+5V" (at 82.55 26.67 0)
+      (effects (font (size 1.27 1.27)))
+    )
+    (property "Footprint" "" (at 82.55 30.48 0)
+      (effects (font (size 1.27 1.27)) hide)
+    )
+    (property "Datasheet" "" (at 82.55 30.48 0)
+      (effects (font (size 1.27 1.27)) hide)
+    )
+    (pin "1")
+    (instances
+      (project "HuntsmanElite"
+        (path "/c8ee06e2-3b90-4589-a28f-453ea39b32a8"
+          (reference "#PWR01") (unit 1)
+        )
+      )
+    )
+  )
+  (symbol (lib_id "power:GND") (at 76.2 125.73 0) (unit 1)
+    (in_bom yes) (on_board yes) (dnp no) (fields_autoplaced)
+    (property "Reference" "#PWR02" (at 76.2 132.08 0)
+      (effects (font (size 1.27 1.27)) hide)
+    )
+    (property "Value" "GND" (at 76.2 130.81 0)
+      (effects (font (size 1.27 1.27)))
+    )
+    (property "Footprint" "" (at 76.2 125.73 0)
+      (effects (font (size 1.27 1.27)) hide)
+    )
+    (property "Datasheet" "" (at 76.2 125.73 0)
+      (effects (font (size 1.27 1.27)) hide)
+    )
+    (pin "1")
+    (instances
+      (project "HuntsmanElite"
+        (path "/c8ee06e2-3b90-4589-a28f-453ea39b32a8"
+          (reference "#PWR02") (unit 1)
+        )
+      )
